Commit message: 暂存gazebo

File: src/probot_fr5_description/urdf/fairino5_v6.urdf (robot description, URDF)
Before this commit: robot fairino5_v6_robot, 7 links, 6 joints
Links:
- link base_link: geometry collision mesh filename=package://probot_fr5_description/meshes/fairino5_v6/base_li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; visual mesh filename=package://probot_fr5_description/meshes/fairino5_v6/base_li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
- link forearm_link: geometry collision mesh filename=package://probot_fr5_description/meshes/fairino5_v6/forearm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; visual mesh filename=package://probot_fr5_description/meshes/fairino5_v6/forearm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
- link shoulder_link: geometry collision mesh filename=package://probot_fr5_description/meshes/fairino5_v6/shoulde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; visual mesh filename=package://probot_fr5_description/meshes/fairino5_v6/shoulde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
- link upperarm_link: geometry collision mesh filename=package://probot_fr5_description/meshes/fairino5_v6/upperar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; visual mesh filename=package://probot_fr5_description/meshes/fairino5_v6/upperar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
- link wrist1_link: geometry collision mesh filename=package://probot_fr5_description/meshes/fairino5_v6/wrist1_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; visual mesh filename=package://probot_fr5_description/meshes/fairino5_v6/wrist1_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
- link wrist2_link: geometry collision mesh filename=package://probot_fr5_description/meshes/fairino5_v6/wrist2_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; visual mesh filename=package://probot_fr5_description/meshes/fairino5_v6/wrist2_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
- link wrist3_link: geometry collision mesh filename=package://probot_fr5_description/meshes/fairino5_v6/wrist3_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; visual mesh filename=package://probot_fr5_description/meshes/fairino5_v6/wrist3_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

File: src/probot_fr5_moveit_config/config/fairino5_v6_robot.ros2_control.xacro (robot description, xacro)
@@ -2,9 +2,11 @@
 <robot xmlns:xacro="http://www.ros.org/wiki/xacro">
     <xacro:macro name="fairino5_v6_robot_ros2_control" params="name initial_positions_file">
-        <xacro:property name="initial_positions" value="${load_yaml(initial_positions_file)['initial_positions']}"/>
+        <xacro:property name="initial_positions" value="${xacro.load_yaml(initial_positions_file)['initial_positions']}"/>
         <ros2_control name="${name}" type="system">
             <hardware>
                 <!-- By default, set up controllers for simulation. This won't work on real hardware -->
-                <plugin>mock_components/GenericSystem</plugin>
+                <!-- <plugin>mock_components/GenericSystem</plugin> -->
+                <!-- gazebo 仿真 -->
+                <plugin>gazebo_ros2_control/GazeboSystem</plugin>
             </hardware>
             <joint name="j1">

File: src/probot_fr5_moveit_config/config/fairino5_v6_robot.urdf.xacro (robot description, xacro)
@@ -2,10 +2,29 @@
 <robot xmlns:xacro="http://www.ros.org/wiki/xacro" name="fairino5_v6_robot">
     <xacro:arg name="initial_positions_file" default="initial_positions.yaml" />
-    <!-- Import fairino5_v6_robot urdf file -->
+    <!-- 默认false，不调用gazebo -->
+    <xacro:arg name="use_sim" default="false" />
+    <!-- Import base URDF -->
     <xacro:include filename="$(find probot_fr5_description)/urdf/fairino5_v6.urdf" />
     <!-- Import control_xacro -->
-    <xacro:include filename="fairino5_v6_robot.ros2_control.xacro" />
+    <xacro:include filename="$(find probot_fr5_moveit_config)/config/fairino5_v6_robot.ros2_control.xacro" />
     <!-- 引入按摩头 -->
-    <xacro:include filename="massage_head.xacro" />
-    <xacro:fairino5_v6_robot_ros2_control name="FakeSystem" initial_positions_file="$(arg initial_positions_file)"/>
+    <xacro:include filename="$(find probot_fr5_moveit_config)/config/massage_head.xacro" />
+    <!-- use_sim 为true时，导入gazebo_ros2_control -->
+    <xacro:if value="$(arg use_sim)">
+        <gazebo>
+        <plugin name="gazebo_ros2_control" filename="libgazebo_ros2_control.so">
+            <parameters>$(find probot_fr5_gazebo)/config/ros2_controllers.yaml</parameters>
+        </plugin>
+        </gazebo>
+    </xacro:if>
+    <!--use_sim 为true时，例化 ros2_control-->
+    <xacro:if value="$(arg use_sim)">
+        <xacro:fairino5_v6_robot_ros2_control name="GazeboSystem"
+        initial_positions_file="$(arg initial_positions_file)"/>
+    </xacro:if>
+    <!--use_sim 为false时，仅在rviz中-->
+    <xacro:unless value="$(arg use_sim)">
+        <xacro:fairino5_v6_robot_ros2_control name="FakeSystem"
+        initial_positions_file="$(arg initial_positions_file)"/>
+    </xacro:unless>
 </robot>
